File: Stubborness.kicad_sch (KiCad schematic)
At the start: 24 parts, among them SW1 SW_Push, U1 ATmega32U4-A, Y1 16MHz

Commit message: Gerber Final, The final steps to the start of the real project.
Created the Gerber files to upload to the manufacturer and test to see if the boards actually work. after this I can start designing my own board in a very long and drawn out process.
Parts:
- R1, R2: value R_Small -> 22
Connections:
- net COL0: now also U1.27 (PD7)
- net COL1: now also U1.28 (PB4)
- net ROW0: now also U1.29 (PB5)
- net ROW1: now also U1.30 (PB6)
Changed lines of the file:
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@@
+    )
+  )
+  (global_label "ROW1" (shape input) (at 149.86 63.5 0) (fields_autoplaced)
+    (effects (font (size 1.27 1.27)) (justify left))
+    (property "Intersheet References" "${INTERSHEET_REFS}" (id 0) (at 157.5345 63.4206 0)
+      (effects (font (size 1.27 1.27)) (justify left) hide)
+    )
+  )
+  (global_label "COL0" (shape input) (at 149.86 96.52 0) (fields_autoplaced)
+    (effects (font (size 1.27 1.27)) (justify left))
+    (property "Intersheet References" "${INTERSHEET_REFS}" (id 0) (at 157.1112 96.4406 0)
+      (effects (font (size 1.27 1.27)) (justify left) hide)
     )
   )
@@
     )
   )
+  (global_label "ROW0" (shape input) (at 149.86 60.96 0) (fields_autoplaced)
+    (effects (font (size 1.27 1.27)) (justify left))
+    (property "Intersheet References" "${INTERSHEET_REFS}" (id 0) (at 157.5345 60.8806 0)
+      (effects (font (size 1.27 1.27)) (justify left) hide)
+    )
+  )
   (global_label "COL0" (shape input) (at 237.49 63.5 90) (fields_autoplaced)
     (effects (font (size 1.27 1.27)) (justify left))
@@
     )
   )
+  (global_label "COL1" (shape input) (at 149.86 58.42 0) (fields_autoplaced)
+    (effects (font (size 1.27 1.27)) (justify left))
+    (property "Intersheet References" "${INTERSHEET_REFS}" (id 0) (at 157.1112 58.3406 0)
+      (effects (font (size 1.27 1.27)) (justify left) hide)
+    )
+  )
   (global_label "D-" (shape input) (at 198.12 40.64 0) (fields_autoplaced)
     (effects (font (size 1.27 1.27)) (justify left))
@@
     (in_bom yes) (on_board yes) (fields_autoplaced)
     (property "Reference" "R1" (id 0) (at 90.17 69.85 90))
-    (property "Value" "R_Small" (id 1) (at 90.17 72.39 90))
+    (property "Value" "22" (id 1) (at 90.17 72.39 90))
     (property "Footprint" "Resistor_SMD:R_0805_2012Metric" (id 2) (at 90.17 76.2 0)
       (effects (font (size 1.27 1.27)) hide)
@@
     (in_bom yes) (on_board yes) (fields_autoplaced)
     (property "Reference" "R2" (id 0) (at 102.87 67.31 90))
-    (property "Value" "R_Small" (id 1) (at 102.87 69.85 90))
+    (property "Value" "22" (id 1) (at 102.87 69.85 90))
     (property "Footprint" "Resistor_SMD:R_0805_2012Metric" (id 2) (at 102.87 73.66 0)
       (effects (font (size 1.27 1.27)) hide)
@@
     )
     (path "/2ebc05ec-a1c0-4787-815c-93f0f44097a2"
-      (reference "R1") (unit 1) (value "R_Small") (footprint "Resistor_SMD:R_0805_2012Metric")
+      (reference "R1") (unit 1) (value "22") (footprint "Resistor_SMD:R_0805_2012Metric")
     )
     (path "/ca855049-e052-48b4-92bf-27eff4b3d72c"
-      (reference "R2") (unit 1) (value "R_Small") (footprint "Resistor_SMD:R_0805_2012Metric")
+      (reference "R2") (unit 1) (value "22") (footprint "Resistor_SMD:R_0805_2012Metric")
     )
     (path "/68a2fd27-1368-41e5-8c42-4933234766d2"
